File: KiCAD/magic-keys.kicad_pcb (KiCad board)
At the start: 2 copper layers, 295.3 x 157.2 mm, 156 parts, among them J1 Keyswitch, K1 Keyswitch, M1 Keyswitch, P1 Keyswitch, Q1 Keyswitch, T1 Keyswitch, U1 Raspberry_Pi_Pico, U2 Keyswitch, X1 Keyswitch, Y1 Keyswitch

Commit message: changed layout for stabs (to be keys), finished schematics
Parts:
- removed OptionDiode2: Diode, ScottoKeebs_Components:Diode_DO-35
- added Backspace2: Keyswitch, ScottoKeebs_Hotswap:Hotswap_Choc_V1_1.00u, F.Cu at (276.2, 76.2)
- added BackspaceDiode2: Diode, ScottoKeebs_Components:Diode_DO-35, B.Cu at (285.8, 84.8)
- added Del2: Keyswitch, ScottoKeebs_Hotswap:Hotswap_Choc_V1_1.00u, F.Cu at (276.2, 57.1)
- added DelDiode2: Diode, ScottoKeebs_Components:Diode_DO-35, B.Cu at (285.8, 65.7)
- added Enter2: Keyswitch, ScottoKeebs_Hotswap:Hotswap_Choc_V1_1.25u, F.Cu at (274.0, 114.3)
- added EnterDiode2: Diode, ScottoKeebs_Components:Diode_DO-35, B.Cu at (283.4, 120.5)
- added Shift3: Keyswitch, ScottoKeebs_Hotswap:Hotswap_Choc_V1_1.50u, F.Cu at (38.0, 132.9)
- added Shift4: Keyswitch, ScottoKeebs_Hotswap:Hotswap_Choc_V1_1.00u, F.Cu at (276.2, 133.3)
- added ShiftDiode3: Diode, ScottoKeebs_Components:Diode_DO-35, B.Cu at (47.6, 139.5)
- added ShiftDiode4: Diode, ScottoKeebs_Components:Diode_DO-35, B.Cu at (285.8, 139.5)
- added Space2: Keyswitch, ScottoKeebs_Hotswap:Hotswap_Choc_V1_1.50u, F.Cu at (119.1, 152.4)
- added Space3: Keyswitch, ScottoKeebs_Hotswap:Hotswap_Choc_V1_1.50u, F.Cu at (147.6, 152.4)
- added Space4: Keyswitch, ScottoKeebs_Hotswap:Hotswap_Choc_V1_1.50u, F.Cu at (176.2, 152.4)
- added SpaceDiode2: Diode, ScottoKeebs_Components:Diode_DO-35, B.Cu at (128.6, 159.5)
- added SpaceDiode3: Diode, ScottoKeebs_Components:Diode_DO-35, B.Cu at (157.2, 160.0)
- added SpaceDiode4: Diode, ScottoKeebs_Components:Diode_DO-35, B.Cu at (185.7, 161.0)
- '"1, -_1, /1, 0)1, 1!1, 2@1, 3#1, 4$1, 5%1, 6^1, 7&1, 8*1, 9(1, ;:1, <,1, =+1, >.1, A1, B1, C1, Cmd1, Cmd2, Control1, D1, Down1, E1, F1, F10, F11, F12, F13, F2, F3, F4, F5, F6, F7, F8, F9, Fn1, G1, H1, I1, J1, K1, L1, Left1, M1, N1, O1, Option1, P1, Q1, R1, Right1, S1, T1, U2, Up1, V1, W1, X1, Y1, Z1, [{1, ]}1, `~1: footprint ScottoKeebs_Hotswap:Hotswap_Choc_V1V2_1.00u -> ScottoKeebs_Hotswap:Hotswap_Choc_V1_1.00u
- Backspace1: footprint ScottoKeebs_Hotswap:Hotswap_Choc_V1V2_2.00u -> ScottoKeebs_Hotswap:Hotswap_Choc_V1_1.00u
- CapsLock1: footprint ScottoKeebs_Hotswap:Hotswap_Choc_V1V2_1.75u -> ScottoKeebs_Hotswap:Hotswap_Choc_V1_1.75u
- Del1, Esc1: footprint ScottoKeebs_Hotswap:Hotswap_Choc_V1V2_1.50u -> ScottoKeebs_Hotswap:Hotswap_Choc_V1_1.00u
- Enter1: footprint ScottoKeebs_Hotswap:Hotswap_Choc_V1V2_2.25u -> ScottoKeebs_Hotswap:Hotswap_Choc_V1_1.00u
- Shift1: footprint ScottoKeebs_Hotswap:Hotswap_Choc_V1V2_2.75u -> ScottoKeebs_Hotswap:Hotswap_Choc_V1_1.25u
- Shift2: footprint ScottoKeebs_Hotswap:Hotswap_Choc_V1V2_2.25u -> ScottoKeebs_Hotswap:Hotswap_Choc_V1_1.25u
- Space1: footprint ScottoKeebs_Hotswap:Hotswap_Choc_V1V2_5.50u -> ScottoKeebs_Hotswap:Hotswap_Choc_V1_1.50u
- Tab1, \|1: footprint ScottoKeebs_Hotswap:Hotswap_Choc_V1V2_1.50u -> ScottoKeebs_Hotswap:Hotswap_Choc_V1_1.50u
- moved UpDiode1 406.9 mm to (266.7, 161.0), turned to 90 degrees
- moved RightDiode1 403.5 mm to (285.8, 159.5), turned to 90 degrees
- moved \|Diode1 396.4 mm to (282.4, 103.8), turned to 90 degrees
- moved ShiftDiode2 373.6 mm to (264.3, 139.5), turned to 90 degrees
- moved ]}Diode1 370.6 mm to (257.0, 103.2), turned to 90 degrees
- moved LeftDiode1 364.5 mm to (228.6, 161.0), turned to 90 degrees
- moved [{Diode1 353.7 mm to (238.0, 103.2), turned to 90 degrees
- moved BackspaceDiode1 351.8 mm to (266.7, 84.3), turned to 90 degrees
- moved DownDiode1 349.9 mm to (247.7, 161.0), turned to 90 degrees
- moved EnterDiode1 347.4 mm to (261.9, 120.5), turned to 90 degrees
- moved DelDiode1 342.7 mm to (266.7, 64.3), turned to 90 degrees
- moved F12Diode1 340.8 mm to (247.8, 64.5), turned to 90 degrees
- moved /?Diode1 340.3 mm to (242.6, 140.2), turned to 90 degrees
- moved >.Diode1 336.2 mm to (223.6, 140.1), turned to 90 degrees
- moved '"Diode1 335.4 mm to (242.9, 121.1), turned to 90 degrees
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Connections:
- U1 pad 26: unconnected-(U1-GPIO20-Pad26) -> Column 14
Routing:
- net Row 5: track 0.00 -> 877.1 mm, vias 0 -> 5
- net Row 4: track 0.00 -> 844.4 mm, vias 0 -> 4
- net Column 12: track 0.00 -> 523.4 mm, vias 0 -> 5
- net Column 1: track 0.00 -> 419.3 mm, vias 0 -> 1
- net Column 0: track 0.00 -> 406.8 mm, vias 0 -> 1
- net Column 2: track 0.00 -> 397.1 mm, vias 0 -> 1
- net Row 3: track 0.00 -> 391.0 mm, vias 0 -> 2
- net Row 2: track 0.00 -> 382.8 mm, vias 0 -> 2
- net Row 1: track 0.00 -> 381.9 mm
- net Column 3: track 0.00 -> 378.7 mm
- net Column 4: track 0.00 -> 371.6 mm
- net Column 5: track 0.00 -> 368.7 mm, vias 0 -> 2
- net Row 0: track 0.00 -> 353.6 mm
- net Column 6: track 0.00 -> 312.4 mm
- net Column 7: track 0.00 -> 305.5 mm, vias 0 -> 2
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Other:
- board size 295.3 x 157.2 mm -> 292.9 x 152.4 mm
- board text added: "@advaitconty"
- board text added: "Orpheus Pico • RP2024 • Hack Club"

Commit message: Optimised wiring
Parts:
- moved CmdDiode2 0.75 mm to (209.5, 161.2)
Connections:
- /1 pad 1: Column 10 -> Column 11
- <,1 pad 1: Column 8 -> Column 9
- >.1 pad 1: Column 9 -> Column 10
- B1 pad 1: Column 5 -> Column 6
- C1 pad 1: Column 3 -> Column 4
- Cmd2 pad 1: Column 5 -> Column 8
- Down1 pad 1: Column 8 -> Column 10
- Left1 pad 1: Column 7 -> Column 9
- M1 pad 1: Column 7 -> Column 8
- N1 pad 1: Column 6 -> Column 7
- Right1 pad 1: Column 10 -> Column 12
- Shift2 pad 1: Column 11 -> Column 12
- Shift3 pad 1: Column 12 -> Column 1
- Space2 pad 1: Column 6 -> Column 5
- Space3 pad 1: Column 11 -> Column 6
- Space4 pad 1: Column 12 -> Column 7
- U1 pad 19: Row 0 -> Column 14
- U1 pad 20: Row 1 -> unconnected-(U1-GPIO15-Pad20)
- U1 pad 21: Row 2 -> Row 0
- U1 pad 22: Row 3 -> Row 1
- U1 pad 24: Row 4 -> Row 2
- U1 pad 25: Row 5 -> Row 3
- U1 pad 26: Column 14 -> Row 4
- U1 pad 27: unconnected-(U1-GPIO21-Pad27) -> Row 5
- Up1 pad 1: Column 9 -> Column 11
- V1 pad 1: Column 4 -> Column 5
- X1 pad 1: Column 2 -> Column 3
- Z1 pad 1: Column 1 -> Column 2
Routing:
- net Row 5: track 877.1 -> 431.0 mm, vias 5 -> 0
- net Row 4: track 844.4 -> 406.4 mm, vias 4 -> 2
- net Column 12: track 523.4 -> 170.0 mm, vias 5 -> 1
- net Column 11: track 275.7 -> 189.2 mm, vias 4 -> 1
- net Column 5: track 368.7 -> 301.5 mm, vias 2 -> 1
- net Column 4: track 371.6 -> 328.5 mm, vias 0 -> 3
- net Column 1: track 419.3 -> 379.6 mm, vias 1 -> 3
- net Column 14: track 50.5 -> 86.9 mm, vias 0 -> 3
- net Column 7: track 305.5 -> 270.3 mm, vias 2 -> 1
- net Column 2: track 397.1 -> 363.7 mm
- net Column 3: track 378.7 -> 351.2 mm, vias 0 -> 3
- net Column 6: track 312.4 -> 286.8 mm, vias 0 -> 1
- net Row 3: track 391.0 -> 366.7 mm, vias 2 -> 3
- net Row 1: track 381.9 -> 357.8 mm
- net Column 10: track 230.8 -> 207.4 mm, vias 2 -> 1
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
Commit message: added mount pounts, added case
Parts:
- added REF**: MountingHole_2.2mm_M2, MountingHole:MountingHole_2.2mm_M2, F.Cu at (4.00, 165.0)
- added REF**: MountingHole_2.2mm_M2, MountingHole:MountingHole_2.2mm_M2, F.Cu at (223.0, 16.0)
- added REF**: MountingHole_2.2mm_M2, MountingHole:MountingHole_2.2mm_M2, F.Cu at (223.0, 38.0)
- added REF**: MountingHole_2.2mm_M2, MountingHole:MountingHole_2.2mm_M2, F.Cu at (4.00, 38.0)
- added REF**: MountingHole_2.2mm_M2, MountingHole:MountingHole_2.2mm_M2, F.Cu at (287.0, 165.0)
- added REF**: MountingHole_2.2mm_M2, MountingHole:MountingHole_2.2mm_M2, F.Cu at (143.0, 165.0)
- added REF**: MountingHole_2.2mm_M2, MountingHole:MountingHole_2.2mm_M2, F.Cu at (125.9, 38.0)
- added REF**: MountingHole_2.2mm_M2, MountingHole:MountingHole_2.2mm_M2, F.Cu at (287.0, 16.0)
Other:
- board size 292.9 x 152.4 mm -> 296 x 162 mm
- board text added: "Noir Keyboard Pro"
- board text added: "can run doom!"
- board text added: "more info about this at https://github.com/advaitconty/noir-keyboard-pro"
- board text added: "powered by hack club"
- board text removed: "@advaitconty"

Commit message: forgot to commit updated PCB
Parts:
- moved REF** 4.92 mm to (282.5, 14.0)
- moved REF** 2.83 mm to (221.0, 14.0)
- moved REF** 2.00 mm to (221.0, 38.0)
- moved REF** 0.71 mm to (3.50, 165.5)
- moved REF** 0.50 mm to (287.5, 165.0)
Routing:
- net Net-(CmdDiode2-A): track 0.00 -> 5.38 mm
- net Net-(SpaceDiode4-A): track 0.00 -> 5.18 mm
- net Net-(LeftDiode1-A): track 0.00 -> 5.18 mm
- net Net-(DownDiode1-A): track 0.00 -> 5.18 mm
- net Row 5: track 431.0 -> 426.3 mm
- net Net-(LDiode1-A): track 0.00 -> 3.37 mm
- net Net-(KDiode1-A): track 0.00 -> 3.37 mm
- net Net-(JDiode1-A): track 0.00 -> 3.37 mm
- net Net-(;:Diode1-A): track 0.00 -> 3.37 mm
- net Net-(NDiode1-A): track 0.00 -> 3.30 mm
- net Net-(<,Diode1-A): track 0.00 -> 3.30 mm
- net Net-(MDiode1-A): track 0.00 -> 3.30 mm
- net Net-(>.Diode1-A): track 0.00 -> 3.27 mm
- net Row 2: track 364.4 -> 363.6 mm
Other:
- board size 296 x 162 mm -> 293 x 160.5 mm

Commit message: added OLED screengit status
Parts:
- added J2: OLED_128x32, ScottoKeebs_Components:OLED_128x32, F.Cu at (7.79, 35.0)
Connections:
- U1 pad 18: unconnected-(U1-GND-Pad18) -> Net-(J2-GND)
- U1 pad 29: unconnected-(U1-GPIO22-Pad29) -> Net-(J2-SCL)
- U1 pad 31: unconnected-(U1-GPIO26_ADC0-Pad31) -> Net-(J2-SDA)
- U1 pad 36: unconnected-(U1-3V3-Pad36) -> Net-(J2-VCC)
Routing:
- net Net-(J2-VCC): track 0.00 -> 285.3 mm, vias 0 -> 1
- net Net-(J2-SCL): track 0.00 -> 275.6 mm, vias 0 -> 1
- net Net-(J2-SDA): track 0.00 -> 274.0 mm, vias 0 -> 1
- net Net-(J2-GND): track 0.00 -> 269.2 mm, vias 0 -> 1
