File: KiCAD/magic-keys.kicad_pcb (KiCad board)
At the start: 2 copper layers, 293 x 160.5 mm, 180 parts, among them J1 Keyswitch, J2 OLED_128x32, K1 Keyswitch, M1 Keyswitch, P1 Keyswitch, Q1 Keyswitch, T1 Keyswitch, U1 Raspberry_Pi_Pico, U2 Keyswitch, X1 Keyswitch, Y1 Keyswitch

Commit message: updated BOM, retraced PCB for a nicer thing
Parts:
- Angle bracket: renamed from >.1
- Blank Backspace: renamed from Backspace1
- Blank Delete: renamed from Del1
- Blank Enter: renamed from Enter1
- Blank Shift: renamed from Shift2
- Blank Shift: renamed from Shift3
- Caps Lock: renamed from CapsLock1
- Closed Sq. Bracket: renamed from ]}1
- Down Arrow: renamed from Down1
- Left Arrow: renamed from Left1
- Open Sq. Bracket: renamed from [{1
- Up Arrow: renamed from Up1
- moved EnterDiode1 0.83 mm to (261.9, 121.3)
- renumbered A1 to A, Option1 to Alt/Option, B1 to B, \|1 to Backslash, Backspace2 to Backspace, C1 to C, <,1 to Chevron, Control1 to Control, D1 to D, -_1 to Dash, Del2 to Delete, E1 to E, 8*1 to Eight, Enter2 to Enter, =+1 to Equals, Esc1 to Escape, F13 to F, 5%1 to Five, 4$1 to Four, Fn1 to Function, G1 to G, H1 to H, I1 to I, J1 to J, K1 to K, L1 to L, M1 to M, N1 to N, 9(1 to Nine, O1 to O, 1!1 to One, P1 to P, Q1 to Q, '"1 to Quotes, R1 to R, Right1 to Right, S1 to S, ;:1 to Semi-Colon, 7&1 to Seven, Shift1 to Shift, Shift4 to Shift, 6^1 to Six, /1 to Slash, Space3 to Space, Space4 to Space, Space1 to Space, Space2 to Space, Cmd1 to Super/Command, Cmd2 to Super/Command, T1 to T, Tab1 to Tab, 3#1 to Three, `~1 to Tilde, 2@1 to Two, U2 to U, V1 to V, W1 to W, X1 to X, Y1 to Y, Z1 to Z, 0)1 to Zero
Connections:
- U1 pad 18: Net-(J2-GND) -> unconnected-(U1-GND-Pad18)
- U1 pad 28: unconnected-(U1-GND-Pad28) -> Net-(J2-GND)
Routing:
- net Net-(J2-GND): track 269.2 -> 251.2 mm
- net Column 1: track 379.6 -> 393.1 mm, vias 3 -> 0
- net Row 1: track 357.8 -> 370.9 mm, vias 0 -> 2
- net Column 13: track 137.2 -> 148.7 mm, vias 3 -> 0
- net Row 0: track 342.2 -> 353.2 mm, vias 4 -> 0
- net Column 6: track 286.8 -> 276.4 mm, vias 1 -> 0
- net Column 0: track 399.9 -> 409.0 mm, vias 5 -> 0
- net Column 10: track 207.4 -> 198.3 mm, vias 1 -> 0
- net Column 9: track 232.7 -> 223.7 mm, vias 1 -> 0
- net Row 2: track 363.6 -> 354.9 mm
- net Column 11: track 189.2 -> 181.1 mm, vias 1 -> 0
- net Column 2: track 363.7 -> 371.3 mm, vias 1 -> 0
- net Column 7: track 270.3 -> 262.8 mm, vias 1 -> 0
- net Column 8: track 252.9 -> 248.2 mm, vias 1 -> 0
- net Column 5: track 301.5 -> 296.9 mm, vias 1 -> 0
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- added copper zone on B.Cu, net (none)
- added copper zone on F.Cu, net (none)
Other:
- board text added: "For more information, visit github.com/advaitconty/noir-keyboard-pro"
- board text added: "Made by advaitconty"
- board text added: "Powered by Hack Club"
- board text added: "Powered by RP2040"
- board text added: "Powered by a Pico controller"
- board text added: "Status OLED"
- board text removed: "Orpheus Pico • RP2024 • Hack Club"
- board text removed: "can run doom!"
- board text removed: "more info about this at https://github.com/advaitconty/noir-keyboard-pro"
- board text removed: "powered by hack club"
